Commit message: corrected the gazebo plugins name

File: src/space_rover_description/urdf/arm.xacro (robot description, xacro)
@@ -99,5 +99,5 @@
 					rpy="0 0 0"/>
 			<geometry>
-				<mesh filename="package://space_rover_description/meshes/arm_02_fixed.dae" scale="${scale_XYZ} ${scale_XYZ} ${scale_XYZ}"/>
+				<box size="${arm_02_X*scale_XYZ} ${arm_02_Y*scale_XYZ} ${arm_02_Z*scale_XYZ}"/>
 			</geometry>
 		</collision>

Commit message: corrected arm from falling

File: src/space_rover_description/urdf/arm.xacro (robot description, xacro)
@@ -52,11 +52,8 @@
 		</inertial>
 	</link>
-  	<joint name="arm_01_joint" type="revolute">
+  	<joint name="arm_01_joint" type="fixed">
 		<parent link="chassis_to_arm_01"/>
 		<child link="arm_01"/>
 		<origin xyz="0 0 0" rpy="0 0 0"/>
-		<limit lower="${-arm_01_limit}" upper="${arm_01_limit}" effort="10000.0" velocity="100.0"/>
-        <axis xyz="0 0 1"/>
-        <joint_properties damping="0.0" friction="0.0"/>
 	</joint>
     <transmission name="arm_01_trans">
@@ -120,11 +117,8 @@
 		</inertial>
 	</link>
-  	<joint name="arm_02_joint" type="revolute">
+  	<joint name="arm_02_joint" type="fixed">
 		<parent link="arm_01_to_arm_02"/>
 		<child link="arm_02"/>
 		<origin xyz="0 0 0" rpy="0 0 0"/>
-		<limit lower="${-arm_02_limit}" upper="${arm_02_limit}" effort="10000.0" velocity="100.0"/>
-        <axis xyz="1 0 0"/>
-        <joint_properties damping="0.0" friction="0.0"/>
 	</joint>
     <transmission name="arm_02_trans">
@@ -188,11 +182,8 @@
 		</inertial>
 	</link>
-  	<joint name="arm_03_joint" type="revolute">
+  	<joint name="arm_03_joint" type="fixed">
 		<parent link="arm_02_to_arm_03"/>
 		<child link="arm_03"/>
 		<origin xyz="0 0 0" rpy="0 0 0"/>
-		<limit lower="${-arm_03_limit}" upper="${arm_03_limit}" effort="10000.0" velocity="100.0"/>
-        <axis xyz="1 0 0"/>
-        <joint_properties damping="0.0" friction="0.0"/>
 	</joint>
     <transmission name="arm_03_trans">
@@ -256,11 +247,8 @@
 		</inertial>
 	</link>
-  	<joint name="arm_04_joint" type="revolute">
+  	<joint name="arm_04_joint" type="fixed">
 		<parent link="arm_03_to_arm_04"/>
 		<child link="arm_04"/>
 		<origin xyz="0 0 0" rpy="0 0 0"/>
-		<limit lower="${-arm_04_limit}" upper="${arm_04_limit}" effort="10000.0" velocity="100.0"/>
-        <axis xyz="0 1 0"/>
-        <joint_properties damping="0.0" friction="0.0"/>
 	</joint>
     <transmission name="arm_04_trans">
@@ -324,11 +312,8 @@
 		</inertial>
 	</link>
-  	<joint name="arm_tools_joint" type="continuous">
+  	<joint name="arm_tools_joint" type="fixed">
 		<parent link="arm_04_to_arm_tools"/>
 		<child link="arm_tools"/>
 		<origin xyz="0 0 0" rpy="0 0 0"/>
-		<limit effort="10000.0" velocity="100.0"/>
-        <axis xyz="0 0 1"/>
-        <joint_properties damping="0.0" friction="0.0"/>
 	</joint>
     <transmission name="arm_tools_trans">
