Commit message: corrected the falling of camera

File: src/space_rover_description/urdf/sensor_mast.xacro (robot description, xacro)
@@ -52,11 +52,8 @@
 		</inertial>
 	</link>
-  	<joint name="mast_p_joint" type="revolute">
+  	<joint name="mast_p_joint" type="fixed">
 		<parent link="chassis_to_mast_p"/>
 		<child link="mast_p"/>
 		<origin xyz="0 0 0" rpy="0 0 0"/>
-		<limit lower="${mast_p_lower_limit}" upper="${mast_p_upper_limit}" effort="10000.0" velocity="100.0"/>
-        <axis xyz="0 1 0"/>
-        <joint_properties damping="0.0" friction="0.0"/>
 	</joint>
     <transmission name="mast_p_trans">
@@ -188,11 +185,8 @@
 		</inertial>
 	</link>
-  	<joint name="mast_cameras_joint" type="revolute">
+  	<joint name="mast_cameras_joint" type="fixed">
 		<parent link="mast_02_to_mast_cameras"/>
 		<child link="mast_cameras"/>
 		<origin xyz="0 0 0" rpy="0 0 0"/>
-		<limit lower="${-mast_cameras_limit}" upper="${mast_cameras_limit}" effort="10000.0" velocity="100.0"/>
-        <axis xyz="1 0 0"/>
-        <joint_properties damping="0.0" friction="0.0"/>
 	</joint>
     <transmission name="mast_02_trans">

Commit message: Added correct position for the camera_link

File: src/space_rover_description/urdf/sensor_mast.xacro (robot description, xacro)
@@ -117,11 +117,8 @@
 		</inertial>
 	</link>
-  	<joint name="mast_02_joint" type="continuous">
+  	<joint name="mast_02_joint" type="fixed">
 		<parent link="mast_p_to_mast_02"/>
 		<child link="mast_02"/>
 		<origin xyz="0 0 0" rpy="0 0 0"/>
-		<limit effort="10000.0" velocity="100.0"/>
-        <axis xyz="0 0 1"/>
-        <joint_properties damping="0.0" friction="0.0"/>
 	</joint>
     <transmission name="mast_02_trans">
@@ -218,12 +215,12 @@
         </visual>
 	</link>
+	<joint name="head_camera_joint" type="fixed">
+        <parent link="mast_cameras"/>
+        <child link="camera_link"/>
+        <origin xyz="0.0 -0.15 0.3" rpy="0 0 -2.4"/>
+    </joint>
     <gazebo reference="camera_link">
         <material>Gazebo/Green</material>
     </gazebo>
-    <joint name="head_camera_joint" type="fixed">
-        <parent link="mast_cameras"/>
-        <child link="camera_link"/>
-        <origin xyz="0.13642 -0.218683 0.222314" rpy="0 0 ${PI}"/>
-    </joint>
   </xacro:macro>
 </robot>
